Commit message: FIX Modify parameters to cope with semi autonomous manipulation
Signed-off-by: Luiz Ricardo Douat <LuizRicardo.Doaut@de.bosch.com>

File: uuv_manipulators/oberon7/oberon7_description/urdf/serial_arm.xacro (robot description, xacro)
@@ -216,5 +216,4 @@
             <origin xyz="0 0 0.31595760629823427" rpy="${-0.5*PI} ${-0.5*PI} 0"/>
             <axis xyz="0 0 1"/>
-            <!-- <dynamics damping="50" friction="200"/> -->
             <dynamics damping="10" friction="10"/>
             <!-- <limit lower="${-90 * d2r}" upper="${90 * d2r}" velocity=".26" effort="200"/> -->
