Commit message: FIX Improving parameters for semi-autonomous manipulation
Signed-off-by: Luiz Ricardo Douat <LuizRicardo.Doaut@de.bosch.com>

File: uuv_manipulators/oberon7/oberon7_description/urdf/parallel_gripper.xacro (robot description, xacro)
@@ -69,5 +69,5 @@
         <origin xyz="0.0444267 0.0391376 0" rpy="0 0 0"/>
         <axis xyz="0 0 1"/>
-        <dynamics damping="5" friction="10"/>
+        <dynamics damping="5" friction="15"/>
         <limit effort="${gripper_effort}" lower="0" upper="${PI*0.3333}" velocity="${gripper_velocity}"/>
     </joint>
@@ -128,5 +128,5 @@
         <origin xyz="0.0444267 -0.0391376 0" rpy="${PI} ${PI} ${PI}"/>
         <axis xyz="0 0 -1"/>
-        <dynamics damping="5" friction="10"/>
+        <dynamics damping="5" friction="15"/>
         <limit effort="${gripper_effort}" lower="0" upper="${PI*0.3333}" velocity="${gripper_velocity}"/>
     </joint>

Commit message: FIX Minor parameter tuning for semi-autonomous manipulation task
Signed-off-by: Luiz Ricardo Douat <LuizRicardo.Doaut@de.bosch.com>

File: uuv_manipulators/oberon7/oberon7_description/urdf/parallel_gripper.xacro (robot description, xacro)
@@ -69,5 +69,5 @@
         <origin xyz="0.0444267 0.0391376 0" rpy="0 0 0"/>
         <axis xyz="0 0 1"/>
-        <dynamics damping="5" friction="15"/>
+        <dynamics damping="5" friction="10"/>
         <limit effort="${gripper_effort}" lower="0" upper="${PI*0.3333}" velocity="${gripper_velocity}"/>
     </joint>
@@ -128,5 +128,5 @@
         <origin xyz="0.0444267 -0.0391376 0" rpy="${PI} ${PI} ${PI}"/>
         <axis xyz="0 0 -1"/>
-        <dynamics damping="5" friction="15"/>
+        <dynamics damping="5" friction="10"/>
         <limit effort="${gripper_effort}" lower="0" upper="${PI*0.3333}" velocity="${gripper_velocity}"/>
     </joint>
